Commit message: update run mapping for scan topic

File: install/hiep_robot2/share/hiep_robot2/urdf/mech/mecanum_wheel.urdf.xacro (robot description, xacro)
@@ -12,5 +12,5 @@
         <origin xyz="0 0 0" rpy="${pi/2} 0 0"/>
         <geometry>
-          <mesh filename="file://$(find mec_mobile_description)/meshes/robot_3d/visual/${side}_wheel_X3.STL"/>
+          <mesh filename="file://$(find hiep_robot2)/meshes/robot_3d/visual/${side}_wheel_X3.STL"/>
         </geometry>
         <material name="dark_gray">

File: install/hiep_robot2/share/hiep_robot2/urdf/robots/robot_3d.urdf.xacro (robot description, xacro)
@@ -5,10 +5,10 @@
     <xacro:arg name="prefix" default=""/>
     <xacro:arg name="use_gazebo" default="false"/>
-    <xacro:include filename="$(find mec_mobile_description)/urdf/mech/robot_3d_base.urdf.xacro"/>
-    <xacro:include filename="$(find mec_mobile_description)/urdf/mech/mecanum_wheel.urdf.xacro"/>
-    <xacro:include filename="$(find mec_mobile_description)/urdf/sensors/rgbd_camera.urdf.xacro"/>
-    <xacro:include filename="$(find mec_mobile_description)/urdf/sensors/lidar.urdf.xacro"/>
-    <xacro:include filename="$(find mec_mobile_description)/urdf/sensors/imu.urdf.xacro"/>
-    <xacro:include filename="$(find mec_mobile_description)/urdf/control/mec_mobile.gazebo"/>
+    <xacro:include filename="$(find hiep_robot2)/urdf/mech/robot_3d_base.urdf.xacro"/>
+    <xacro:include filename="$(find hiep_robot2)/urdf/mech/mecanum_wheel.urdf.xacro"/>
+    <xacro:include filename="$(find hiep_robot2)/urdf/sensors/rgbd_camera.urdf.xacro"/>
+    <xacro:include filename="$(find hiep_robot2)/urdf/sensors/lidar.urdf.xacro"/>
+    <xacro:include filename="$(find hiep_robot2)/urdf/sensors/imu.urdf.xacro"/>
+    <xacro:include filename="$(find hiep_robot2)/urdf/control/mec_mobile.gazebo"/>
     <xacro:robot_3d_base prefix="$(arg prefix)"/>
     <xacro:mecanum_wheel

File: src/hiep_robot2/urdf/robots/robot_3d.urdf.xacro (robot description, xacro)
@@ -153,3 +153,9 @@
     </link>
     <!-- 2.5.1 End -->
+<link name="base_footprint"/>
+<joint name="base_footprint_joint" type="fixed">
+  <parent link="base_footprint"/>
+  <child link="base_link"/>
+  <origin xyz="0 0 0" rpy="0 0 0"/>
+</joint>
 </robot>
